File: RPI_Cam3_RL.kicad_sch (KiCad schematic)
At the start: 42 parts, among them J1 in, Q1 2N7002, U1 RPI_CAM_3

Commit message: Updated Pcb Design -Small Radius
Connections:
- net +5V: now also J1.1 (Pin_1); no longer J1.3 (Pin_3)
- net GND: now also J1.3 (Pin_3); no longer J1.1 (Pin_1)
Changed lines of the file:
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@@
 	)
 	(junction
+		(at 31.75 40.64)
+		(diameter 0)
+		(color 0 0 0 0)
+	)
+	(junction
 		(at 100.33 43.18)
 		(diameter 0)
@@
 	)
 	(junction
+		(at 31.7288 45.72)
+		(diameter 0)
+		(color 0 0 0 0)
+	)
+	(junction
 		(at 100.33 77.47)
 		(diameter 0)
@@
 	(wire
 		(pts
+			(xy 31.7288 45.72) (xy 39.37 45.72)
+		)
+		(stroke
+			(width 0)
+			(type default)
+		)
+	)
+	(wire
+		(pts
 			(xy 214.63 92.71) (xy 214.63 114.3)
 		)
@@
 	(wire
 		(pts
-			(xy 27.94 45.72) (xy 39.37 45.72)
+			(xy 27.94 45.72) (xy 31.7288 45.72)
 		)
 		(stroke
@@
 	(wire
 		(pts
+			(xy 31.75 40.64) (xy 39.37 40.64)
+		)
+		(stroke
+			(width 0)
+			(type default)
+		)
+	)
+	(wire
+		(pts
 			(xy 59.69 96.52) (xy 59.69 100.33)
 		)
@@
 	(wire
 		(pts
-			(xy 27.94 40.64) (xy 39.37 40.64)
+			(xy 27.94 40.64) (xy 31.75 40.64)
 		)
 		(stroke
@@
 	)
 	(symbol
+		(lib_id "power:PWR_FLAG")
+		(at 31.7288 45.72 180)
+		(unit 1)
+		(exclude_from_sim no)
+		(in_bom yes)
+		(on_board yes)
+		(dnp no)
+		(fields_autoplaced yes)
+		(property "Reference" "#FLG02"
+			(at 31.7288 47.625 0)
+			(effects
+				(font
+					(size 1.27 1.27)
+				)
+				(hide yes)
+			)
+		)
+		(property "Value" "PWR_FLAG"
+			(at 31.7288 50.8 0)
+			(effects
+				(font
+					(size 1.27 1.27)
+				)
+			)
+		)
+		(property "Footprint" ""
+			(at 31.7288 45.72 0)
+			(effects
+				(font
+					(size 1.27 1.27)
+				)
+				(hide yes)
+			)
+		)
+		(property "Datasheet" "~"
+			(at 31.7288 45.72 0)
+			(effects
+				(font
+					(size 1.27 1.27)
+				)
+				(hide yes)
+			)
+		)
+		(property "Description" "Special symbol for telling ERC where power comes from"
+			(at 31.7288 45.72 0)
+			(effects
+				(font
+					(size 1.27 1.27)
+				)
+				(hide yes)
+			)
+		)
+		(pin "1"
+		)
+		(instances
+			(project "RPI_Cam3_RL"
+				(path "/53c6947d-8834-4e12-a59f-ee14606a4e52"
+					(reference "#FLG02")
+					(unit 1)
+				)
+			)
+		)
+	)
+	(symbol
 		(lib_id "Mechanical:MountingHole")
 		(at 266.7 63.5 0)
@@
 	(symbol
 		(lib_id "power:+5V")
-		(at 39.37 40.64 0)
+		(at 39.37 45.72 180)
 		(unit 1)
 		(exclude_from_sim no)
@@
 		(fields_autoplaced yes)
 		(property "Reference" "#PWR01"
-			(at 39.37 44.45 0)
+			(at 39.37 41.91 0)
 			(effects
 				(font
@@
 		)
 		(property "Value" "+5V"
-			(at 39.37 35.56 0)
+			(at 39.37 50.8 0)
 			(effects
 				(font
@@
 		)
 		(property "Footprint" ""
-			(at 39.37 40.64 0)
+			(at 39.37 45.72 0)
 			(effects
 				(font
@@
 		)
 		(property "Datasheet" ""
-			(at 39.37 40.64 0)
+			(at 39.37 45.72 0)
 			(effects
 				(font
@@
 		)
 		(property "Description" "Power symbol creates a global label with name \"+5V\""
-			(at 39.37 40.64 0)
+			(at 39.37 45.72 0)
 			(effects
 				(font
@@
 	)
 	(symbol
+		(lib_id "power:PWR_FLAG")
+		(at 31.75 40.64 0)
+		(unit 1)
+		(exclude_from_sim no)
+		(in_bom yes)
+		(on_board yes)
+		(dnp no)
+		(fields_autoplaced yes)
+		(property "Reference" "#FLG01"
+			(at 31.75 38.735 0)
+			(effects
+				(font
+					(size 1.27 1.27)
+				)
+				(hide yes)
+			)
+		)
+		(property "Value" "PWR_FLAG"
+			(at 31.75 35.56 0)
+			(effects
+				(font
+					(size 1.27 1.27)
+				)
+			)
+		)
+		(property "Footprint" ""
+			(at 31.75 40.64 0)
+			(effects
+				(font
+					(size 1.27 1.27)
+				)
+				(hide yes)
+			)
+		)
+		(property "Datasheet" "~"
+			(at 31.75 40.64 0)
+			(effects
+				(font
+					(size 1.27 1.27)
+				)
+				(hide yes)
+			)
+		)
+		(property "Description" "Special symbol for telling ERC where power comes from"
+			(at 31.75 40.64 0)
+			(effects
+				(font
+					(size 1.27 1.27)
+				)
+				(hide yes)
+			)
+		)
+		(pin "1"
+		)
+		(instances
+			(project ""
+				(path "/53c6947d-8834-4e12-a59f-ee14606a4e52"
+					(reference "#FLG01")
+					(unit 1)
+				)
+			)
+		)
+	)
+	(symbol
 		(lib_id "Mechanical:MountingHole")
 		(at 266.7 49.53 0)
@@
 	(symbol
 		(lib_id "power:GND")
-		(at 39.37 45.72 0)
+		(at 39.37 40.64 180)
 		(unit 1)
 		(exclude_from_sim no)
@@
 		(fields_autoplaced yes)
 		(property "Reference" "#PWR02"
-			(at 39.37 52.07 0)
+			(at 39.37 34.29 0)
 			(effects
 				(font
@@
 		)
 		(property "Value" "GND"
-			(at 39.37 50.8 0)
+			(at 39.37 35.56 0)
 			(effects
 				(font
@@
 		)
 		(property "Footprint" ""
-			(at 39.37 45.72 0)
+			(at 39.37 40.64 0)
 			(effects
 				(font
@@
 		)
 		(property "Datasheet" ""
-			(at 39.37 45.72 0)
+			(at 39.37 40.64 0)
 			(effects
 				(font
@@
 		)
 		(property "Description" "Power symbol creates a global label with name \"GND\" , ground"
-			(at 39.37 45.72 0)
+			(at 39.37 40.64 0)
 			(effects
 				(font

Commit message: design updates
Parts:
- added H10, H9: m2, MountingHole:MountingHole_3.2mm_M3, symbol Mechanical:MountingHole
Changed lines of the file:
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@@
+	(symbol
+		(lib_id "Mechanical:MountingHole")
+		(at 237.49 132.08 0)
+		(unit 1)
+		(exclude_from_sim no)
+		(in_bom no)
+		(on_board yes)
+		(dnp no)
+		(fields_autoplaced yes)
+		(property "Reference" "H9"
+			(at 240.03 130.8099 0)
+			(effects
+				(font
+					(size 1.27 1.27)
+				)
+				(justify left)
+			)
+		)
+		(property "Value" "m2"
+			(at 240.03 133.3499 0)
+			(effects
+				(font
+					(size 1.27 1.27)
+				)
+				(justify left)
+			)
+		)
+		(property "Footprint" "MountingHole:MountingHole_3.2mm_M3"
+			(at 237.49 132.08 0)
+			(effects
+				(font
+					(size 1.27 1.27)
+				)
+				(hide yes)
+			)
+		)
+		(property "Datasheet" "~"
+			(at 237.49 132.08 0)
+			(effects
+				(font
+					(size 1.27 1.27)
+				)
+				(hide yes)
+			)
+		)
+		(property "Description" "Mounting Hole without connection"
+			(at 237.49 132.08 0)
+			(effects
+				(font
+					(size 1.27 1.27)
+				)
+				(hide yes)
+			)
+		)
+		(instances
+			(project "RPI_Cam3_RL"
+				(path "/53c6947d-8834-4e12-a59f-ee14606a4e52"
+					(reference "H9")
+					(unit 1)
+				)
+			)
+		)
+	)
 	(symbol
 		(lib_id "Mechanical:MountingHole")
@@
 					(unit 1)
 				)
+			)
+		)
+	)
+	(symbol
+		(lib_id "Mechanical:MountingHole")
+		(at 264.16 132.08 0)
+		(unit 1)
+		(exclude_from_sim no)
+		(in_bom no)
+		(on_board yes)
+		(dnp no)
+		(fields_autoplaced yes)
+		(property "Reference" "H10"
+			(at 266.7 130.8099 0)
+			(effects
+				(font
+					(size 1.27 1.27)
+				)
+				(justify left)
+			)
+		)
+		(property "Value" "m2"
+			(at 266.7 133.3499 0)
+			(effects
+				(font
+					(size 1.27 1.27)
+				)
+				(justify left)
+			)
+		)
+		(property "Footprint" "MountingHole:MountingHole_3.2mm_M3"
+			(at 264.16 132.08 0)
+			(effects
+				(font
+					(size 1.27 1.27)
+				)
+				(hide yes)
+			)
+		)
+		(property "Datasheet" "~"
+			(at 264.16 132.08 0)
+			(effects
+				(font
+					(size 1.27 1.27)
+				)
+				(hide yes)
+			)
+		)
+		(property "Description" "Mounting Hole without connection"
+			(at 264.16 132.08 0)
+			(effects
+				(font
+					(size 1.27 1.27)
+				)
+				(hide yes)
+			)
+		)
+		(instances
+			(project "RPI_Cam3_RL"
+				(path "/53c6947d-8834-4e12-a59f-ee14606a4e52"
+					(reference "H10")
+					(unit 1)
+				)

Commit message: silkscreen updates
Other:
- company: (none) -> Delta Things
- title: (none) -> RPI_CAM_RingLight
Changed lines of the file:
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@@
 	(generator_version "9.0")
 	(paper "A4")
+	(title_block
+		(title "RPI_CAM_RingLight")
+		(date "2026-01-07")
+		(rev "1.0.0")
+		(company "Delta Things")
+		(comment 1 "Mount for official Raspberry Pi Cameras")
+	)
 	(junction
 		(at 100.33 92.71)
